File: stm32l053.sch (KiCad schematic (older format))
At the start: 13 parts, among them U1 STM32_LQFP64

Commit message: 10uF cap
Parts:
- added C4: 10uF, Capacitors_SMD:C_0805_HandSoldering, symbol C
- gave numbers to parts that had none: 11
Connections:
- net Earth: now also C4.2
- net VDD: now also C4.1
Changed lines of the file:
@@
 $EndComp
 $Comp
-L Earth #PWR01
+L Earth #PWR16
 U 1 1 58021BE1
 P 9650 1350
-F 0 "#PWR01" H 9650 1100 50  0001 C CNN
+F 0 "#PWR16" H 9650 1100 50  0001 C CNN
 F 1 "Earth" H 9650 1200 50  0001 C CNN
 F 2 "" H 9650 1350 50  0000 C CNN
@@
 $EndComp
 $Comp
-L VDD #PWR03
+L VDD #PWR15
 U 1 1 58021C2A
 P 9650 1050
-F 0 "#PWR03" H 9650 900 50  0001 C CNN
+F 0 "#PWR15" H 9650 900 50  0001 C CNN
 F 1 "VDD" H 9650 1200 50  0000 C CNN
 F 2 "" H 9650 1050 50  0000 C CNN
@@
 $EndComp
 $Comp
-L GNDA #PWR05
+L GNDA #PWR11
 U 1 1 58021F75
 P 7050 6200
-F 0 "#PWR05" H 7050 5950 50  0001 C CNN
+F 0 "#PWR11" H 7050 5950 50  0001 C CNN
 F 1 "GNDA" H 7050 6050 50  0000 C CNN
 F 2 "" H 7050 6200 50  0000 C CNN
@@
 $EndComp
 $Comp
-L Earth #PWR06
+L Earth #PWR14
 U 1 1 58021F89
 P 7550 6200
-F 0 "#PWR06" H 7550 5950 50  0001 C CNN
+F 0 "#PWR14" H 7550 5950 50  0001 C CNN
 F 1 "Earth" H 7550 6050 50  0001 C CNN
 F 2 "" H 7550 6200 50  0000 C CNN
@@
 $EndComp
 $Comp
-L GNDA #PWR07
+L GNDA #PWR10
 U 1 1 58022154
 P 7050 5700
-F 0 "#PWR07" H 7050 5450 50  0001 C CNN
+F 0 "#PWR10" H 7050 5450 50  0001 C CNN
 F 1 "GNDA" H 7050 5550 50  0000 C CNN
 F 2 "" H 7050 5700 50  0000 C CNN
@@
 $EndComp
 $Comp
-L Earth #PWR08
+L Earth #PWR13
 U 1 1 580221FA
 P 7550 5700
-F 0 "#PWR08" H 7550 5450 50  0001 C CNN
+F 0 "#PWR13" H 7550 5450 50  0001 C CNN
 F 1 "Earth" H 7550 5550 50  0001 C CNN
 F 2 "" H 7550 5700 50  0000 C CNN
@@
 $EndComp
 $Comp
-L VDD #PWR010
+L VDD #PWR12
 U 1 1 5802295B
 P 7350 950
-F 0 "#PWR010" H 7350 800 50  0001 C CNN
+F 0 "#PWR12" H 7350 800 50  0001 C CNN
 F 1 "VDD" H 7350 1100 50  0000 C CNN
 F 2 "" H 7350 950 50  0000 C CNN
@@
 $EndComp
 $Comp
-L Earth #PWR011
+L Earth #PWR7
 U 1 1 5802320E
 P 5600 4700
-F 0 "#PWR011" H 5600 4450 50  0001 C CNN
+F 0 "#PWR7" H 5600 4450 50  0001 C CNN
 F 1 "Earth" H 5600 4550 50  0001 C CNN
 F 2 "" H 5600 4700 50  0000 C CNN
@@
 $EndComp
 $Comp
-L C C?
+L C C3
 U 1 1 58032557
 P 6950 1650
-F 0 "C?" V 7100 1600 50  0000 L CNN
+F 0 "C3" V 7100 1600 50  0000 L CNN
 F 1 "100nF" V 6800 1550 50  0000 L CNN
 F 2 "" H 6988 1500 50  0000 C CNN
@@
 $EndComp
 $Comp
-L R R?
+L R R2
 U 1 1 58032944
 P 7100 1450
-F 0 "R?" V 7180 1450 50  0000 C CNN
+F 0 "R2" V 7180 1450 50  0000 C CNN
 F 1 "0" V 7100 1450 50  0000 C CNN
 F 2 "" V 7030 1450 50  0000 C CNN
@@
 $EndComp
 $Comp
-L Earth #PWR?
+L Earth #PWR9
 U 1 1 5803310F
 P 6700 1700
-F 0 "#PWR?" H 6700 1450 50  0001 C CNN
+F 0 "#PWR9" H 6700 1450 50  0001 C CNN
 F 1 "Earth" H 6700 1550 50  0001 C CNN
 F 2 "" H 6700 1700 50  0000 C CNN
@@
 If USB is not used this\npin must be tied to VDD .
 $Comp
-L R R?
+L R R3
 U 1 1 5803422C
 P 7800 1450
-F 0 "R?" V 7880 1450 50  0000 C CNN
+F 0 "R3" V 7880 1450 50  0000 C CNN
 F 1 "0" V 7800 1450 50  0000 C CNN
 F 2 "" V 7730 1450 50  0000 C CNN
@@
 MCO
 $Comp
-L C C?
+L C C2
 U 1 1 58034E62
 P 6500 5150
-F 0 "C?" H 6525 5250 50  0000 L CNN
+F 0 "C2" H 6525 5250 50  0000 L CNN
 F 1 "C" H 6525 5050 50  0000 L CNN
 F 2 "" H 6538 5000 50  0000 C CNN
@@
 $EndComp
 $Comp
-L Earth #PWR?
+L Earth #PWR8
 U 1 1 58034EA2
 P 6500 5300
-F 0 "#PWR?" H 6500 5050 50  0001 C CNN
+F 0 "#PWR8" H 6500 5050 50  0001 C CNN
 F 1 "Earth" H 6500 5150 50  0001 C CNN
 F 2 "" H 6500 5300 50  0000 C CNN
@@
 $EndComp
 $Comp
-L CONN_01X06 P?
+L CONN_01X06 P1
 U 1 1 58036840
 P 1700 1400
-F 0 "P?" H 1700 1750 50  0000 C CNN
+F 0 "P1" H 1700 1750 50  0000 C CNN
 F 1 "SWD" V 1800 1400 50  0000 C CNN
 F 2 "" H 1700 1400 50  0000 C CNN
@@
 $EndComp
 $Comp
-L Earth #PWR?
+L Earth #PWR4
 U 1 1 580369A9
 P 2400 1350
-F 0 "#PWR?" H 2400 1100 50  0001 C CNN
+F 0 "#PWR4" H 2400 1100 50  0001 C CNN
 F 1 "Earth" H 2400 1200 50  0001 C CNN
 F 2 "" H 2400 1350 50  0000 C CNN
@@
 SWO
 $Comp
-L VDD #PWR?
+L VDD #PWR3
 U 1 1 5803734F
 P 1900 1150
-F 0 "#PWR?" H 1900 1000 50  0001 C CNN
+F 0 "#PWR3" H 1900 1000 50  0001 C CNN
 F 1 "VDD" H 1900 1300 50  0000 C CNN
 F 2 "" H 1900 1150 50  0000 C CNN
@@
 $EndComp
 $Comp
-L R R?
+L R R1
 U 1 1 58037533
 P 5600 4550
-F 0 "R?" V 5680 4550 50  0000 C CNN
+F 0 "R1" V 5680 4550 50  0000 C CNN
 F 1 "10K" V 5600 4550 50  0000 C CNN
 F 2 "" V 5530 4550 50  0000 C CNN
@@
 OSC32_OUT
 $Comp
-L CONN_01X02 P?
+L CONN_01X02 P5
 U 1 1 58037B90
 P 6250 7150
-F 0 "P?" H 6250 7300 50  0000 C CNN
+F 0 "P5" H 6250 7300 50  0000 C CNN
 F 1 "Ext Xtal" V 6350 7150 50  0000 C CNN
 F 2 "" H 6250 7150 50  0000 C CNN
@@
 PD2
 $Comp
-L Earth #PWR?
+L Earth #PWR2
 U 1 1 5803DE21
 P 1500 4700
-F 0 "#PWR?" H 1500 4450 50  0001 C CNN
+F 0 "#PWR2" H 1500 4450 50  0001 C CNN
 F 1 "Earth" H 1500 4550 50  0001 C CNN
 F 2 "" H 1500 4700 50  0000 C CNN
@@
 $EndComp
 $Comp
-L VDD #PWR?
+L VDD #PWR1
 U 1 1 5803DE79
 P 1500 2500
-F 0 "#PWR?" H 1500 2350 50  0001 C CNN
+F 0 "#PWR1" H 1500 2350 50  0001 C CNN
 F 1 "VDD" H 1500 2650 50  0000 C CNN
 F 2 "" H 1500 2500 50  0000 C CNN
@@
 $EndComp
 $Comp
-L CONN_01X23 P?
+L CONN_01X23 P2
 U 1 1 5803E207
 P 1700 3600
-F 0 "P?" H 1700 4800 50  0000 C CNN
+F 0 "P2" H 1700 4800 50  0000 C CNN
 F 1 "CONN_01X23" V 1800 3600 50  0000 C CNN
 F 2 "" H 1700 3600 50  0000 C CNN
@@
 $EndComp
 $Comp
-L CONN_01X23 P?
+L CONN_01X23 P3
 U 1 1 5803E381
 P 2450 3600
-F 0 "P?" H 2450 4800 50  0000 C CNN
+F 0 "P3" H 2450 4800 50  0000 C CNN
 F 1 "CONN_01X23" V 2550 3600 50  0000 C CNN
 F 2 "" H 2450 3600 50  0000 C CNN
@@
 	3000 4700 2650 4700
 $Comp
-L CONN_01X02 P?
+L CONN_01X02 P4
 U 1 1 5803EC4A
 P 3900 1350
-F 0 "P?" H 3900 1500 50  0000 C CNN
+F 0 "P4" H 3900 1500 50  0000 C CNN
 F 1 "BOOT_MODE" V 4000 1350 50  0000 C CNN
 F 2 "" H 3900 1350 50  0000 C CNN
@@
 BOOT0
 $Comp
-L VDD #PWR?
+L VDD #PWR6
 U 1 1 5803ED1E
 P 3700 1300
-F 0 "#PWR?" H 3700 1150 50  0001 C CNN
+F 0 "#PWR6" H 3700 1150 50  0001 C CNN
 F 1 "VDD" H 3700 1450 50  0000 C CNN
 F 2 "" H 3700 1300 50  0000 C CNN
@@
 $EndComp
 $Comp
-L SW_PUSH SW?
+L SW_PUSH SW1
 U 1 1 5803EFB1
 P 3650 1900
-F 0 "SW?" H 3800 2010 50  0000 C CNN
+F 0 "SW1" H 3800 2010 50  0000 C CNN
 F 1 "SW_PUSH" H 3650 1820 50  0000 C CNN
 F 2 "" H 3650 1900 50  0000 C CNN
@@
 $EndComp
 $Comp
-L Earth #PWR?
+L Earth #PWR5
 U 1 1 5803F003
 P 3350 1900
-F 0 "#PWR?" H 3350 1650 50  0001 C CNN
+F 0 "#PWR5" H 3350 1650 50  0001 C CNN
 F 1 "Earth" H 3350 1750 50  0001 C CNN
 F 2 "" H 3350 1900 50  0000 C CNN
@@
 Text GLabel 3950 1900 2    60   Input ~ 0
 NRST
+$Comp
+L Earth #PWR18
+U 1 1 58039244
+P 10100 1350
+F 0 "#PWR18" H 10100 1100 50  0001 C CNN
+F 1 "Earth" H 10100 1200 50  0001 C CNN
+F 2 "" H 10100 1350 50  0000 C CNN
+F 3 "" H 10100 1350 50  0000 C CNN
+	1    10100 1350
+	1    0    0    -1
+$EndComp
+$Comp
+L VDD #PWR17
+U 1 1 5803924A
+P 10100 1050
+F 0 "#PWR17" H 10100 900 50  0001 C CNN
+F 1 "VDD" H 10100 1200 50  0000 C CNN
+F 2 "" H 10100 1050 50  0000 C CNN
+F 3 "" H 10100 1050 50  0000 C CNN
+	1    10100 1050
+	1    0    0    -1
+$EndComp
+$Comp
+L C C4
+U 1 1 58039250
+P 10100 1200
+F 0 "C4" H 10125 1300 50  0000 L CNN
+F 1 "10uF" H 10125 1100 50  0000 L CNN
+F 2 "Capacitors_SMD:C_0805_HandSoldering" H 10138 1050 50  0001 C CNN
+F 3 "" H 10100 1200 50  0000 C CNN
+	1    10100 1200
+	1    0    0    -1
+$EndComp
 $EndSCHEMATC

Commit message: Restart layout
Parts:
- C2, C3: footprint (none) -> Capacitors_SMD:C_0805_HandSoldering
- P1: footprint (none) -> Pin_Headers:Pin_Header_Straight_1x06
- P2, P3: footprint (none) -> Pin_Headers:Pin_Header_Straight_1x23
- P4: footprint (none) -> Pin_Headers:Pin_Header_Straight_1x02
- P5, R1, R2, R3: footprint (none) -> Resistors_SMD:R_0805_HandSoldering
- SW1: footprint (none) -> Buttons_Switches_SMD:SW_SPST_B3U-1000P
Changed lines of the file:
@@
 $EndComp
 $Comp
-L Earth #PWR16
+L Earth #PWR01
 U 1 1 58021BE1
 P 9650 1350
-F 0 "#PWR16" H 9650 1100 50  0001 C CNN
+F 0 "#PWR01" H 9650 1100 50  0001 C CNN
 F 1 "Earth" H 9650 1200 50  0001 C CNN
 F 2 "" H 9650 1350 50  0000 C CNN
@@
 $EndComp
 $Comp
-L VDD #PWR15
+L VDD #PWR02
 U 1 1 58021C2A
 P 9650 1050
-F 0 "#PWR15" H 9650 900 50  0001 C CNN
+F 0 "#PWR02" H 9650 900 50  0001 C CNN
 F 1 "VDD" H 9650 1200 50  0000 C CNN
 F 2 "" H 9650 1050 50  0000 C CNN
@@
 $EndComp
 $Comp
-L GNDA #PWR11
+L GNDA #PWR03
 U 1 1 58021F75
 P 7050 6200
-F 0 "#PWR11" H 7050 5950 50  0001 C CNN
+F 0 "#PWR03" H 7050 5950 50  0001 C CNN
 F 1 "GNDA" H 7050 6050 50  0000 C CNN
 F 2 "" H 7050 6200 50  0000 C CNN
@@
 $EndComp
 $Comp
-L Earth #PWR14
+L Earth #PWR04
 U 1 1 58021F89
 P 7550 6200
-F 0 "#PWR14" H 7550 5950 50  0001 C CNN
+F 0 "#PWR04" H 7550 5950 50  0001 C CNN
 F 1 "Earth" H 7550 6050 50  0001 C CNN
 F 2 "" H 7550 6200 50  0000 C CNN
@@
 $EndComp
 $Comp
-L GNDA #PWR10
+L GNDA #PWR05
 U 1 1 58022154
 P 7050 5700
-F 0 "#PWR10" H 7050 5450 50  0001 C CNN
+F 0 "#PWR05" H 7050 5450 50  0001 C CNN
 F 1 "GNDA" H 7050 5550 50  0000 C CNN
 F 2 "" H 7050 5700 50  0000 C CNN
@@
 $EndComp
 $Comp
-L Earth #PWR13
+L Earth #PWR06
 U 1 1 580221FA
 P 7550 5700
-F 0 "#PWR13" H 7550 5450 50  0001 C CNN
+F 0 "#PWR06" H 7550 5450 50  0001 C CNN
 F 1 "Earth" H 7550 5550 50  0001 C CNN
 F 2 "" H 7550 5700 50  0000 C CNN
@@
 $EndComp
 $Comp
-L VDD #PWR12
+L VDD #PWR07
 U 1 1 5802295B
 P 7350 950
-F 0 "#PWR12" H 7350 800 50  0001 C CNN
+F 0 "#PWR07" H 7350 800 50  0001 C CNN
 F 1 "VDD" H 7350 1100 50  0000 C CNN
 F 2 "" H 7350 950 50  0000 C CNN
@@
 $EndComp
 $Comp
-L Earth #PWR7
+L Earth #PWR08
 U 1 1 5802320E
 P 5600 4700
-F 0 "#PWR7" H 5600 4450 50  0001 C CNN
+F 0 "#PWR08" H 5600 4450 50  0001 C CNN
 F 1 "Earth" H 5600 4550 50  0001 C CNN
 F 2 "" H 5600 4700 50  0000 C CNN
@@
 F 0 "C3" V 7100 1600 50  0000 L CNN
 F 1 "100nF" V 6800 1550 50  0000 L CNN
-F 2 "" H 6988 1500 50  0000 C CNN
+F 2 "Capacitors_SMD:C_0805_HandSoldering" H 6988 1500 50  0001 C CNN
 F 3 "" H 6950 1650 50  0000 C CNN
 	1    6950 1650
@@
 F 0 "R2" V 7180 1450 50  0000 C CNN
 F 1 "0" V 7100 1450 50  0000 C CNN
-F 2 "" V 7030 1450 50  0000 C CNN
+F 2 "Resistors_SMD:R_0805_HandSoldering" V 7030 1450 50  0001 C CNN
 F 3 "" H 7100 1450 50  0000 C CNN
 	1    7100 1450
@@
 $EndComp
 $Comp
-L Earth #PWR9
+L Earth #PWR09
 U 1 1 5803310F
 P 6700 1700
-F 0 "#PWR9" H 6700 1450 50  0001 C CNN
+F 0 "#PWR09" H 6700 1450 50  0001 C CNN
 F 1 "Earth" H 6700 1550 50  0001 C CNN
 F 2 "" H 6700 1700 50  0000 C CNN
@@
 F 0 "R3" V 7880 1450 50  0000 C CNN
 F 1 "0" V 7800 1450 50  0000 C CNN
-F 2 "" V 7730 1450 50  0000 C CNN
+F 2 "Resistors_SMD:R_0805_HandSoldering" V 7730 1450 50  0001 C CNN
 F 3 "" H 7800 1450 50  0000 C CNN
 	1    7800 1450
@@
 F 0 "C2" H 6525 5250 50  0000 L CNN
 F 1 "C" H 6525 5050 50  0000 L CNN
-F 2 "" H 6538 5000 50  0000 C CNN
+F 2 "Capacitors_SMD:C_0805_HandSoldering" H 6538 5000 50  0001 C CNN
 F 3 "" H 6500 5150 50  0000 C CNN
 	1    6500 5150
@@
 $EndComp
 $Comp
-L Earth #PWR8
+L Earth #PWR010
 U 1 1 58034EA2
 P 6500 5300
-F 0 "#PWR8" H 6500 5050 50  0001 C CNN
+F 0 "#PWR010" H 6500 5050 50  0001 C CNN
 F 1 "Earth" H 6500 5150 50  0001 C CNN
 F 2 "" H 6500 5300 50  0000 C CNN
@@
 F 0 "P1" H 1700 1750 50  0000 C CNN
 F 1 "SWD" V 1800 1400 50  0000 C CNN
-F 2 "" H 1700 1400 50  0000 C CNN
+F 2 "Pin_Headers:Pin_Header_Straight_1x06" H 1700 1400 50  0001 C CNN
 F 3 "" H 1700 1400 50  0000 C CNN
 	1    1700 1400
@@
 $EndComp
 $Comp
-L Earth #PWR4
+L Earth #PWR011
 U 1 1 580369A9
 P 2400 1350
-F 0 "#PWR4" H 2400 1100 50  0001 C CNN
+F 0 "#PWR011" H 2400 1100 50  0001 C CNN
 F 1 "Earth" H 2400 1200 50  0001 C CNN
 F 2 "" H 2400 1350 50  0000 C CNN
@@
 SWO
 $Comp
-L VDD #PWR3
+L VDD #PWR012
 U 1 1 5803734F
 P 1900 1150
-F 0 "#PWR3" H 1900 1000 50  0001 C CNN
+F 0 "#PWR012" H 1900 1000 50  0001 C CNN
 F 1 "VDD" H 1900 1300 50  0000 C CNN
 F 2 "" H 1900 1150 50  0000 C CNN
@@
 F 0 "R1" V 5680 4550 50  0000 C CNN
 F 1 "10K" V 5600 4550 50  0000 C CNN
-F 2 "" V 5530 4550 50  0000 C CNN
+F 2 "Resistors_SMD:R_0805_HandSoldering" V 5530 4550 50  0001 C CNN
 F 3 "" H 5600 4550 50  0000 C CNN
 	1    5600 4550
@@
 F 0 "P5" H 6250 7300 50  0000 C CNN
 F 1 "Ext Xtal" V 6350 7150 50  0000 C CNN
-F 2 "" H 6250 7150 50  0000 C CNN
+F 2 "Resistors_SMD:R_0805_HandSoldering" H 6250 7150 50  0001 C CNN
 F 3 "" H 6250 7150 50  0000 C CNN
 	1    6250 7150
@@
 PD2
 $Comp
-L Earth #PWR2
+L Earth #PWR013
 U 1 1 5803DE21
 P 1500 4700
-F 0 "#PWR2" H 1500 4450 50  0001 C CNN
+F 0 "#PWR013" H 1500 4450 50  0001 C CNN
 F 1 "Earth" H 1500 4550 50  0001 C CNN
 F 2 "" H 1500 4700 50  0000 C CNN
@@
 $EndComp
 $Comp
-L VDD #PWR1
+L VDD #PWR014
 U 1 1 5803DE79
 P 1500 2500
-F 0 "#PWR1" H 1500 2350 50  0001 C CNN
+F 0 "#PWR014" H 1500 2350 50  0001 C CNN
 F 1 "VDD" H 1500 2650 50  0000 C CNN
 F 2 "" H 1500 2500 50  0000 C CNN
@@
 F 0 "P2" H 1700 4800 50  0000 C CNN
 F 1 "CONN_01X23" V 1800 3600 50  0000 C CNN
-F 2 "" H 1700 3600 50  0000 C CNN
+F 2 "Pin_Headers:Pin_Header_Straight_1x23" H 1700 3600 50  0001 C CNN
 F 3 "" H 1700 3600 50  0000 C CNN
 	1    1700 3600
@@
 F 0 "P3" H 2450 4800 50  0000 C CNN
 F 1 "CONN_01X23" V 2550 3600 50  0000 C CNN
-F 2 "" H 2450 3600 50  0000 C CNN
+F 2 "Pin_Headers:Pin_Header_Straight_1x23" H 2450 3600 50  0001 C CNN
 F 3 "" H 2450 3600 50  0000 C CNN
 	1    2450 3600
@@
 F 0 "P4" H 3900 1500 50  0000 C CNN
 F 1 "BOOT_MODE" V 4000 1350 50  0000 C CNN
-F 2 "" H 3900 1350 50  0000 C CNN
+F 2 "Pin_Headers:Pin_Header_Straight_1x02" H 3900 1350 50  0001 C CNN
 F 3 "" H 3900 1350 50  0000 C CNN
 	1    3900 1350
@@
 BOOT0
 $Comp
-L VDD #PWR6
+L VDD #PWR015
 U 1 1 5803ED1E
 P 3700 1300
-F 0 "#PWR6" H 3700 1150 50  0001 C CNN
+F 0 "#PWR015" H 3700 1150 50  0001 C CNN
 F 1 "VDD" H 3700 1450 50  0000 C CNN
 F 2 "" H 3700 1300 50  0000 C CNN
@@
 F 0 "SW1" H 3800 2010 50  0000 C CNN
 F 1 "SW_PUSH" H 3650 1820 50  0000 C CNN
-F 2 "" H 3650 1900 50  0000 C CNN
+F 2 "Buttons_Switches_SMD:SW_SPST_B3U-1000P" H 3650 1900 50  0001 C CNN
 F 3 "" H 3650 1900 50  0000 C CNN
 	1    3650 1900
@@
 $EndComp
 $Comp
-L Earth #PWR5
+L Earth #PWR016
 U 1 1 5803F003
 P 3350 1900
-F 0 "#PWR5" H 3350 1650 50  0001 C CNN
+F 0 "#PWR016" H 3350 1650 50  0001 C CNN
 F 1 "Earth" H 3350 1750 50  0001 C CNN
 F 2 "" H 3350 1900 50  0000 C CNN
@@
 NRST
 $Comp
-L Earth #PWR18
+L Earth #PWR017
 U 1 1 58039244
 P 10100 1350
-F 0 "#PWR18" H 10100 1100 50  0001 C CNN
+F 0 "#PWR017" H 10100 1100 50  0001 C CNN
 F 1 "Earth" H 10100 1200 50  0001 C CNN
 F 2 "" H 10100 1350 50  0000 C CNN
@@
 $EndComp
 $Comp
-L VDD #PWR17
+L VDD #PWR018
 U 1 1 5803924A
 P 10100 1050
-F 0 "#PWR17" H 10100 900 50  0001 C CNN
+F 0 "#PWR018" H 10100 900 50  0001 C CNN
 F 1 "VDD" H 10100 1200 50  0000 C CNN
 F 2 "" H 10100 1050 50  0000 C CNN
