File: stm32l053.sch (KiCad schematic (older format))
At the start: 14 parts, among them P1 SWD, P2 CONN_01X23, P3 CONN_01X23, P4 BOOT_MODE, P5 Ext Xtal, SW1 SW_PUSH, U1 STM32_LQFP64

Commit message: Design rules
Parts:
- removed P4: BOOT_MODE, Pin_Headers:Pin_Header_Straight_1x02, symbol CONN_01X02
- added C5, C6, C7: 100nF, Capacitors_SMD:C_0805_HandSoldering, symbol C
- added P4: BOOT0, Pin_Headers:Pin_Header_Straight_1x01, symbol CONN_01X01
- P5: footprint Resistors_SMD:R_0805_HandSoldering -> Crystals:Crystal_SMD_0603_2Pads_obsolete
Connections:
- net BOOT0: now also P4.1 (P1)
- net Earth: now also P2.2 (P2), C5.2, C6.2, C7.2; no longer P2.23 (P23)
- net PA0: now also P2.3 (P3); no longer P2.2 (P2)
- net PA1: now also P2.4 (P4); no longer P2.3 (P3)
- net PA10: now also P2.13 (P13); no longer P2.12 (P12)
- net PA11: now also P2.14 (P14); no longer P2.13 (P13)
- net PA12: now also P2.15 (P15); no longer P2.14 (P14)
- net PA15: now also P2.16 (P16); no longer P2.15 (P15)
- net PA2: now also P2.5 (P5); no longer P2.4 (P4)
- net PA3: now also P2.6 (P6); no longer P2.5 (P5)
- net PA4: now also P2.7 (P7); no longer P2.6 (P6)
- net PA5: now also P2.8 (P8); no longer P2.7 (P7)
- net PA6: now also P2.9 (P9); no longer P2.8 (P8)
- net PA7: now also P2.10 (P10); no longer P2.9 (P9)
- net PA8: now also P2.11 (P11); no longer P2.10 (P10)
- net PA9: now also P2.12 (P12); no longer P2.11 (P11)
- net PC0: now also P2.17 (P17); no longer P2.16 (P16)
- net PC1: now also P2.18 (P18); no longer P2.17 (P17)
- net PC2: now also P2.19 (P19); no longer P2.18 (P18)
- net PC3: now also P2.20 (P20); no longer P2.19 (P19)
- net PC4: now also P2.21 (P21); no longer P2.20 (P20)
- net PC5: now also P2.22 (P22); no longer P2.21 (P21)
- net PC6: now also P2.23 (P23); no longer P2.22 (P22)
- net VDD: now also C5.1, C6.1, C7.1
Other:
- moved on the sheet: C4
Changed lines of the file:
@@
 F 0 "P5" H 6250 7300 50  0000 C CNN
 F 1 "Ext Xtal" V 6350 7150 50  0000 C CNN
-F 2 "Resistors_SMD:R_0805_HandSoldering" H 6250 7150 50  0001 C CNN
+F 2 "Crystals:Crystal_SMD_0603_2Pads_obsolete" H 6250 7150 50  0001 C CNN
 F 3 "" H 6250 7150 50  0000 C CNN
 	1    6250 7150
@@
 Wire Wire Line
 	7550 6200 7050 6200
-Text Label 1200 2600 0    60   ~ 0
+Text Label 1200 2700 0    60   ~ 0
 PA0
-Text Label 1200 2700 0    60   ~ 0
+Text Label 1200 2800 0    60   ~ 0
 PA1
-Text Label 1200 2800 0    60   ~ 0
+Text Label 1200 2900 0    60   ~ 0
 PA2
-Text Label 1200 2900 0    60   ~ 0
+Text Label 1200 3000 0    60   ~ 0
 PA3
-Text Label 1200 3000 0    60   ~ 0
+Text Label 1200 3100 0    60   ~ 0
 PA4
-Text Label 1200 3100 0    60   ~ 0
+Text Label 1200 3200 0    60   ~ 0
 PA5
-Text Label 1200 3200 0    60   ~ 0
+Text Label 1200 3300 0    60   ~ 0
 PA6
-Text Label 1200 3300 0    60   ~ 0
+Text Label 1200 3400 0    60   ~ 0
 PA7
-Text Label 1200 3400 0    60   ~ 0
+Text Label 1200 3500 0    60   ~ 0
 PA8
-Text Label 1200 3500 0    60   ~ 0
+Text Label 1200 3600 0    60   ~ 0
 PA9
-Text Label 1200 3600 0    60   ~ 0
+Text Label 1200 3700 0    60   ~ 0
 PA10
-Text Label 1200 3700 0    60   ~ 0
+Text Label 1200 3800 0    60   ~ 0
 PA11
-Text Label 1200 3800 0    60   ~ 0
+Text Label 1200 3900 0    60   ~ 0
 PA12
 Wire Wire Line
+	1200 3900 1500 3900
+Wire Wire Line
 	1200 3800 1500 3800
 Wire Wire Line
@@
 	1200 3300 1500 3300
 Wire Wire Line
-	1200 3200 1500 3200
-Wire Wire Line
-	1500 3100 1200 3100
+	1500 3200 1200 3200
+Wire Wire Line
+	1200 3100 1500 3100
 Wire Wire Line
 	1200 3000 1500 3000
@@
 Wire Wire Line
 	1200 2700 1500 2700
-Wire Wire Line
-	1200 2600 1500 2600
 Text Label 6200 3700 0    60   ~ 0
 PA15
@@
 Wire Wire Line
 	6200 2200 6500 2200
-Text Label 1200 3900 0    60   ~ 0
+Text Label 1200 4000 0    60   ~ 0
 PA15
 Wire Wire Line
-	1200 3900 1500 3900
+	1200 4000 1500 4000
 Text Label 8800 2200 2    60   ~ 0
 PB0
@@
 Wire Wire Line
 	8450 4200 8800 4200
-Text Label 1200 4000 0    60   ~ 0
+Text Label 1200 4100 0    60   ~ 0
 PC0
-Text Label 1200 4100 0    60   ~ 0
+Text Label 1200 4200 0    60   ~ 0
 PC1
-Text Label 1200 4200 0    60   ~ 0
+Text Label 1200 4300 0    60   ~ 0
 PC2
-Text Label 1200 4400 0    60   ~ 0
+Text Label 1200 4500 0    60   ~ 0
 PC4
-Text Label 1200 4500 0    60   ~ 0
+Text Label 1200 4600 0    60   ~ 0
 PC5
-Text Label 1200 4600 0    60   ~ 0
+Text Label 1200 4700 0    60   ~ 0
 PC6
 Text Label 3000 4000 2    60   ~ 0
@@
 Wire Wire Line
 	2650 4600 3000 4600
-Text Label 1200 4300 0    60   ~ 0
+Text Label 1200 4400 0    60   ~ 0
 PC3
 Text Label 6200 3900 0    60   ~ 0
@@
 L Earth #PWR013
 U 1 1 5803DE21
-P 1500 4700
-F 0 "#PWR013" H 1500 4450 50  0001 C CNN
-F 1 "Earth" H 1500 4550 50  0001 C CNN
-F 2 "" H 1500 4700 50  0000 C CNN
-F 3 "" H 1500 4700 50  0000 C CNN
-	1    1500 4700
+P 900 2650
+F 0 "#PWR013" H 900 2400 50  0001 C CNN
+F 1 "Earth" H 900 2500 50  0001 C CNN
+F 2 "" H 900 2650 50  0000 C CNN
+F 3 "" H 900 2650 50  0000 C CNN
+	1    900  2650
 	1    0    0    -1
 $EndComp
@@
 $EndComp
 Wire Wire Line
-	1200 4600 1500 4600
-Wire Wire Line
-	1200 4000 1500 4000
+	1200 4700 1500 4700
 Wire Wire Line
 	1200 4100 1500 4100
@@
 	1200 4200 1500 4200
 Wire Wire Line
-	1500 4300 1200 4300
-Wire Wire Line
-	1200 4400 1500 4400
-Wire Wire Line
-	1500 4500 1200 4500
+	1200 4300 1500 4300
+Wire Wire Line
+	1500 4400 1200 4400
+Wire Wire Line
+	1200 4500 1500 4500
+Wire Wire Line
+	1500 4600 1200 4600
 Wire Wire Line
 	3000 4700 2650 4700
-$Comp
-L CONN_01X02 P4
-U 1 1 5803EC4A
-P 3900 1350
-F 0 "P4" H 3900 1500 50  0000 C CNN
-F 1 "BOOT_MODE" V 4000 1350 50  0000 C CNN
-F 2 "Pin_Headers:Pin_Header_Straight_1x02" H 3900 1350 50  0001 C CNN
-F 3 "" H 3900 1350 50  0000 C CNN
-	1    3900 1350
-	1    0    0    -1
-$EndComp
 Text GLabel 3700 1400 0    60   Input ~ 0
 BOOT0
-$Comp
-L VDD #PWR015
-U 1 1 5803ED1E
-P 3700 1300
-F 0 "#PWR015" H 3700 1150 50  0001 C CNN
-F 1 "VDD" H 3700 1450 50  0000 C CNN
-F 2 "" H 3700 1300 50  0000 C CNN
-F 3 "" H 3700 1300 50  0000 C CNN
-	1    3700 1300
-	1    0    0    -1
-$EndComp
 $Comp
 L SW_PUSH SW1
@@
 $EndComp
 $Comp
-L Earth #PWR016
+L Earth #PWR015
 U 1 1 5803F003
 P 3350 1900
-F 0 "#PWR016" H 3350 1650 50  0001 C CNN
+F 0 "#PWR015" H 3350 1650 50  0001 C CNN
 F 1 "Earth" H 3350 1750 50  0001 C CNN
 F 2 "" H 3350 1900 50  0000 C CNN
@@
 NRST
 $Comp
-L Earth #PWR017
+L Earth #PWR016
 U 1 1 58039244
-P 10100 1350
-F 0 "#PWR017" H 10100 1100 50  0001 C CNN
-F 1 "Earth" H 10100 1200 50  0001 C CNN
-F 2 "" H 10100 1350 50  0000 C CNN
-F 3 "" H 10100 1350 50  0000 C CNN
-	1    10100 1350
-	1    0    0    -1
-$EndComp
-$Comp
-L VDD #PWR018
+P 9650 2100
+F 0 "#PWR016" H 9650 1850 50  0001 C CNN
+F 1 "Earth" H 9650 1950 50  0001 C CNN
+F 2 "" H 9650 2100 50  0000 C CNN
+F 3 "" H 9650 2100 50  0000 C CNN
+	1    9650 2100
+	1    0    0    -1
+$EndComp
+$Comp
+L VDD #PWR017
 U 1 1 5803924A
-P 10100 1050
-F 0 "#PWR018" H 10100 900 50  0001 C CNN
-F 1 "VDD" H 10100 1200 50  0000 C CNN
-F 2 "" H 10100 1050 50  0000 C CNN
-F 3 "" H 10100 1050 50  0000 C CNN
-	1    10100 1050
+P 9650 1800
+F 0 "#PWR017" H 9650 1650 50  0001 C CNN
+F 1 "VDD" H 9650 1950 50  0000 C CNN
+F 2 "" H 9650 1800 50  0000 C CNN
+F 3 "" H 9650 1800 50  0000 C CNN
+	1    9650 1800
 	1    0    0    -1
 $EndComp
@@
 L C C4
 U 1 1 58039250
-P 10100 1200
-F 0 "C4" H 10125 1300 50  0000 L CNN
-F 1 "10uF" H 10125 1100 50  0000 L CNN
-F 2 "Capacitors_SMD:C_0805_HandSoldering" H 10138 1050 50  0001 C CNN
-F 3 "" H 10100 1200 50  0000 C CNN
-	1    10100 1200
-	1    0    0    -1
-$EndComp
+P 9650 1950
+F 0 "C4" H 9675 2050 50  0000 L CNN
+F 1 "10uF" H 9675 1850 50  0000 L CNN
+F 2 "Capacitors_SMD:C_0805_HandSoldering" H 9688 1800 50  0001 C CNN
+F 3 "" H 9650 1950 50  0000 C CNN
+	1    9650 1950
+	1    0    0    -1
+$EndComp
+$Comp
+L CONN_01X01 P4
+U 1 1 5803B76E
+P 3900 1400
+F 0 "P4" H 3900 1500 50  0000 C CNN
+F 1 "BOOT0" V 4000 1400 50  0000 C CNN
+F 2 "Pin_Headers:Pin_Header_Straight_1x01" H 3900 1400 50  0001 C CNN
+F 3 "" H 3900 1400 50  0000 C CNN
+	1    3900 1400
+	1    0    0    -1
+$EndComp
+$Comp
+L C C5
+U 1 1 5803B990
+P 9950 1200
+F 0 "C5" H 9975 1300 50  0000 L CNN
+F 1 "100nF" H 9975 1100 50  0000 L CNN
+F 2 "Capacitors_SMD:C_0805_HandSoldering" H 9988 1050 50  0001 C CNN
+F 3 "" H 9950 1200 50  0000 C CNN
+	1    9950 1200
+	1    0    0    -1
+$EndComp
+$Comp
+L C C6
+U 1 1 5803BA02
+P 10250 1200
+F 0 "C6" H 10275 1300 50  0000 L CNN
+F 1 "100nF" H 10275 1100 50  0000 L CNN
+F 2 "Capacitors_SMD:C_0805_HandSoldering" H 10288 1050 50  0001 C CNN
+F 3 "" H 10250 1200 50  0000 C CNN
+	1    10250 1200
+	1    0    0    -1
+$EndComp
+$Comp
+L C C7
+U 1 1 5803BA4A
+P 10700 1200
+F 0 "C7" H 10725 1300 50  0000 L CNN
+F 1 "100nF" H 10725 1100 50  0000 L CNN
+F 2 "Capacitors_SMD:C_0805_HandSoldering" H 10738 1050 50  0001 C CNN
+F 3 "" H 10700 1200 50  0000 C CNN
+	1    10700 1200
+	1    0    0    -1
+$EndComp
+Wire Wire Line
+	9650 1050 10250 1050
+Connection ~ 9950 1050
+Wire Wire Line
+	9650 1350 10250 1350
+Connection ~ 9950 1350
+$Comp
+L Earth #PWR018
+U 1 1 5803BDC8
+P 10700 1350
+F 0 "#PWR018" H 10700 1100 50  0001 C CNN
+F 1 "Earth" H 10700 1200 50  0001 C CNN
+F 2 "" H 10700 1350 50  0000 C CNN
+F 3 "" H 10700 1350 50  0000 C CNN
+	1    10700 1350
+	1    0    0    -1
+$EndComp
+Text Label 10700 950  0    60   ~ 0
+VDDA
+Wire Wire Line
+	10700 950  10700 1050
+Text Label 7200 1900 1    60   ~ 0
+VDDA
+Wire Wire Line
+	900  2650 900  2600
+Wire Wire Line
+	900  2600 1500 2600
 $EndSCHEMATC
