File: stm32l053.kicad_pcb (KiCad board)
At the start: 2 copper layers, 23.9 x 59.4 mm, 18 parts, among them P1 SWD, P2 CONN_01X23, P3 CONN_01X23, P4 BOOT0, P5 Ext Xtal, P6 MCO, SW1 RESET, U1 STM32_LQFP64

Commit message: Ground plane
Routing:
- added copper zone on B.Cu, net Earth
- added copper zone on F.Cu, net Earth
Changed lines of the file:
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@@
   (segment (start 156.544918 106.788858) (end 157.57398 107.81792) (width 0.254) (layer F.Cu) (net 57))
   (via (at 157.57398 107.81792) (size 0.762) (drill 0.4064) (layers F.Cu B.Cu) (net 57))
+  (zone (net 2) (net_name Earth) (layer F.Cu) (hatch edge 0.508)
+    (connect_pads (clearance 0.508))
+    (min_thickness 0.254)
+    (fill yes (arc_segments 16) (thermal_gap 0.508) (thermal_bridge_width 0.508))
+    (polygon
+      (pts
+        (xy 137.922 79.502) (xy 161.798 79.502) (xy 161.798 138.938) (xy 137.922 138.938)
+      )
+    )
+  )
+  (zone (net 2) (net_name Earth) (layer B.Cu) (hatch edge 0.508)
+    (connect_pads (clearance 0.508))
+    (min_thickness 0.254)
+    (fill yes (arc_segments 16) (thermal_gap 0.508) (thermal_bridge_width 0.508))
+    (polygon
+      (pts
+        (xy 137.922 79.502) (xy 161.798 79.502) (xy 161.798 138.938) (xy 137.922 138.938)
+      )
+    )
+  )
 )
